File: Decoration/Periodt_decoration.kicad_pcb (KiCad board)
At the start: 2 copper layers, 320.9 x 105.2 mm, 5 parts, among them J3 Conn_01x01, J4 Conn_01x01, J5 Conn_01x01, J7 Conn_01x01

Commit message: change keyboard name for Periodt
Parts:
- added J3: Conn_01x01, kbd_Hole:m2_Screw_Hole_EdgeCuts, F.Cu at (341.9, 80.6)
- moved J5 1.00 mm to (341.9, 35.5)
- moved J7 1.00 mm to (341.9, 125.7)
Other:
- board size 320.9 x 105.2 mm -> 321.9 x 105.2 mm
