File: pcb/Periodt.kicad_pcb (KiCad board)
At the start: 2 copper layers, 314.3 x 98.8 mm, 172 parts, among them SW1 SW_PUSH, SW10 SW_PUSH, SW11 SW_PUSH, SW12 SW_PUSH, SW13 SW_PUSH, SW14 SW_PUSH, SW15 SW_PUSH, SW16 SW_PUSH, SW17 SW_PUSH, SW18 SW_PUSH, SW19 SW_PUSH, SW2 SW_PUSH, SW20 SW_PUSH, SW21 SW_PUSH, SW22 SW_PUSH, SW23 SW_PUSH, SW24 SW_PUSH, SW25 SW_PUSH, SW26 SW_PUSH, SW28 SW_PUSH, SW29 SW_PUSH, SW3 SW_PUSH, SW30 SW_PUSH, SW31 SW_PUSH, SW32 SW_PUSH, SW33 SW_PUSH, SW34 SW_PUSH, SW35 SW_PUSH, SW36 SW_PUSH, SW37 SW_PUSH, SW38 SW_PUSH, SW39 SW_PUSH, SW4 RotaryEncoder_Switch, SW40 SW_PUSH, SW41 SW_PUSH, SW42 SW_PUSH, SW43 SW_PUSH, SW44 SW_PUSH, SW45 SW_PUSH, SW46 SW_PUSH, SW47 SW_PUSH, SW48 SW_PUSH, SW49 SW_PUSH, SW5 SW_PUSH, SW50 SW_PUSH, SW51 SW_PUSH, SW52 SW_PUSH, SW53 SW_PUSH, SW54 SW_PUSH, SW55 SW_PUSH, SW56 SW_PUSH, SW57 RotaryEncoder_Switch, SW6 SW_PUSH, SW7 SW_PUSH, SW8 SW_PUSH, SW9 SW_PUSH, U1 rp2040-zero

Commit message: change keyboard name for Periodt
Parts:
- moved G*** 11.5 mm to (118.9, 25.6)
- moved D53 5.07 mm to (284.0, 105.1)
- moved L49 5.02 mm to (278.2, 99.3)
- moved SW53 4.77 mm to (278.0, 104.7)
- moved SW8 4.74 mm to (64.8, 104.7)
- moved L37 4.73 mm to (64.4, 99.2)
- moved D8 4.46 mm to (70.8, 104.2)
Routing:
- net Row3: track 615.8 -> 627.6 mm
- net LEDVCC: track 1400.3 -> 1392.4 mm
- net Net-(L36-DOUT): track 63.2 -> 68.5 mm
- net Net-(L49-DOUT): track 23.4 -> 18.6 mm
- net Net-(L37-DOUT): track 24.3 -> 19.5 mm
- net Col1: track 434.5 -> 439.3 mm
- net Col5: track 437.7 -> 442.3 mm
- net Net-(L48-DOUT): track 63.7 -> 68.3 mm
- net GND: track 1563.9 -> 1567.2 mm
- net Col3: track 428.4 -> 425.7 mm
- net Net-(D8-A): track 6.66 -> 6.16 mm
